Commit message: updated assignment

File: IR_catkin_ws/src/planar2r_description/urdf/planar2r_model.urdf (robot description, URDF)
Before this commit: robot planar2r, 6 links, 6 joints
Links:
- removed link j2
- removed link link1a
Joints:
- removed joint j2_link2
- removed joint l1
- removed joint l2
- joint endEff: origin xyz=0 0 0 -> xyz=${link2_length} 0 0
- joint joint1: child link1a -> link1
- joint joint2: child j2 -> link2; origin xyz=0 0 0 -> xyz=${link1_length} 0 0

File: IR_catkin_ws/src/planar3r_description/urdf/planar3r_model.urdf (robot description, URDF)
Before this commit: robot planar3r, 8 links, 9 joints
Links:
- removed link j2
- removed link j3
- removed link link1a
Joints:
- removed joint j2_link2
- removed joint j3_link3
- removed joint l1
- removed joint l2
- removed joint l3
- joint endEff: origin xyz=0 0 0 -> xyz=${link3_length} 0 0
- joint joint1: child link1a -> link1
- joint joint2: child j2 -> link2; origin xyz=0 0 0 -> xyz=${link1_length} 0 0
- joint joint3: child j3 -> link3; origin xyz=0 0 0 -> xyz=${link2_length} 0 0

File: IR_catkin_ws/src/spatial3r_description/urdf/spatial3r_model.urdf (robot description, URDF)
Before this commit: robot planar3r, 8 links, 9 joints
Links:
- removed link j2
- removed link j3
- removed link link1a
Joints:
- removed joint j2_link2
- removed joint j3_link3
- removed joint l1
- removed joint l2
- removed joint l3
- joint endEff: origin xyz=0 0 0 -> xyz=${link3_length} 0 0
- joint joint1: child link1a -> link1
- joint joint2: child j2 -> link2; origin xyz=0 0 0 rpy=1.570796327 0 0 -> xyz=0 0 ${link1_length} rpy=1.570796327 0 0
- joint joint3: child j3 -> link3; origin xyz=0 0 0 rpy=0 0 0 -> xyz=${link2_length} 0 0 rpy=0 0 0
